File: Design/Pico_Mdot2_r3/P42-Pico_Mdot2_r3.kicad_sch (KiCad schematic)
At the start: 33 parts, among them J1 QWIIC, J2 Bus_M.2_Socket_AE, J3 Micro_SD_Card_Det2, Q1 RJU003N03, U3 LDO-1.1, U4 AP2125KS-1.8, U5 TXS0102DQE, U6 TXS0102DQE

Commit message: Update P42-Pico_Mdot2_r3.kicad_sch
Changed power LEDs to yellow
Parts:
- D1, D2: value Green -> Yellow; JLCPCB # C434420 -> C434424; LCSC Part # C434420 -> C434424; Mfr PN 150060GS75000 -> 150060YS75000; Mfr1 PN SZYY0603G -> SZYY0603Y
Changed lines of the file:
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@@
 			)
 		)
-		(property "Value" "Green"
+		(property "Value" "Yellow"
 			(at 238.76 227.33 90)
 			(effects
@@
 			)
 		)
-		(property "Description" "LED GREEN CLEAR 0603 SMD"
+		(property "Description" "LED YELLOW CLEAR 0603 SMD"
 			(at 237.49 226.06 0)
 			(effects
@@
 			)
 		)
-		(property "Mfr PN" "150060GS75000"
+		(property "Mfr PN" "150060YS75000"
 			(at 237.49 226.06 0)
 			(effects
@@
 			)
 		)
-		(property "Mfr1 PN" "SZYY0603G"
+		(property "Mfr1 PN" "SZYY0603Y"
 			(at 237.49 226.06 0)
 			(effects
@@
 			)
 		)
-		(property "JLCPCB #" "C434420"
+		(property "JLCPCB #" "C434424"
 			(at 237.49 226.06 0)
 			(effects
@@
 			)
 		)
-		(property "LCSC Part #" "C434420"
+		(property "LCSC Part #" "C434424"
 			(at 237.49 226.06 0)
 			(effects
@@
 			)
 		)
-		(property "Value" "Green"
+		(property "Value" "Yellow"
 			(at 257.81 219.71 90)
 			(effects
@@
 			)
 		)
-		(property "Description" "LED GREEN CLEAR 0603 SMD"
+		(property "Description" "LED YELLOW CLEAR 0603 SMD"
 			(at 256.54 218.44 0)
 			(effects
@@
 			)
 		)
-		(property "Mfr PN" "150060GS75000"
+		(property "Mfr PN" "150060YS75000"
 			(at 256.54 218.44 0)
 			(effects
@@
 			)
 		)
-		(property "Mfr1 PN" "SZYY0603G"
+		(property "Mfr1 PN" "SZYY0603Y"
 			(at 256.54 218.44 0)
 			(effects
@@
 			)
 		)
-		(property "JLCPCB #" "C434420"
+		(property "JLCPCB #" "C434424"
 			(at 256.54 218.44 0)
 			(effects
@@
 			)
 		)
-		(property "LCSC Part #" "C434420"
+		(property "LCSC Part #" "C434424"
 			(at 256.54 218.44 0)
 			(effects

Commit message: SCH update with license
.kicad_sch sources and PDF docs.
Parts:
- C13, C22, C23, C8: LCSC Part #2 (none) -> C170151
- FB1: LCSC Part #2 (none) -> C85833
- J2, TP3, TP4, TP5: now left out of the parts list
- J3: Mfr (none) -> Molex; Mfr PN (none) -> 104031-0811
- Q1: LCSC Part #2 (none) -> C308741
Connections:
- net GND: now also D2.1 (K); no longer D1.1 (K)
- net at Q1.3 (D): now also D1.1 (K); no longer D2.1 (K)
Other:
- moved on the sheet: D1, D2, R3, R4
